Commit message: before I integrate two files, I want to set a checkpoint

File: install/cobrotic/share/cobrotic/cobra.urdf (robot description, URDF)
Before this commit: robot cobra, 9 links, 8 joints
Links:
- link arm: geometry visual box size=0.40 0.50 1.60
Joints:
- joint arm_to_forearm: limit lower=0 upper=3.14 effort=1000.0 velocity=0.5 -> lower=0 upper=3.14 effort=1000.0 velocity=1.0; origin xyz=0 0 1.4 rpy=0 2.616 0 -> xyz=0 0 1.2 rpy=0 2.70526034 0
- joint bottom_to_pedestal: limit lower=0.00 upper=3.14 effort=1000.0 velocity=0.5 -> lower=0.00 upper=3.66519143 effort=1000.0 velocity=1.0
- joint left_gripper_joint: limit lower=0 upper=0.523599 effort=1000.0 velocity=0.5 -> lower=0 upper=0.523599 effort=1000.0 velocity=1.0
- joint pedestal_to_arm: limit lower=0 upper=1.91986 effort=1000.0 velocity=0.5 -> lower=0 upper=2.18166157 effort=1000.0 velocity=1.0; origin xyz=0 0 0.3 rpy=0 -0.785398 0 -> xyz=0 0 0.4 rpy=0 -1.13446401 0
- joint right_gripper_joint: limit lower=0.0 upper=0.523599 effort=1000.0 velocity=0.5 -> lower=0.0 upper=0.523599 effort=1000.0 velocity=1.0

File: src/cobrotic/urdf/cobra.urdf (robot description, URDF)
Before this commit: robot cobra, 9 links, 8 joints
Links:
- link arm: geometry visual box size=0.40 0.50 1.60
Joints:
- joint arm_to_forearm: limit lower=0 upper=3.14 effort=1000.0 velocity=0.5 -> lower=0 upper=3.14 effort=1000.0 velocity=1.0; origin xyz=0 0 1.4 rpy=0 2.616 0 -> xyz=0 0 1.2 rpy=0 2.70526034 0
- joint bottom_to_pedestal: limit lower=0.00 upper=3.4906585 effort=1000.0 velocity=0.5 -> lower=0.00 upper=3.66519143 effort=1000.0 velocity=1.0
- joint left_gripper_joint: limit lower=0 upper=0.523599 effort=1000.0 velocity=0.5 -> lower=0 upper=0.523599 effort=1000.0 velocity=1.0
- joint pedestal_to_arm: limit lower=0 upper=1.91986 effort=1000.0 velocity=0.5 -> lower=0 upper=2.18166157 effort=1000.0 velocity=1.0; origin xyz=0 0 0.3 rpy=0 -0.785398 0 -> xyz=0 0 0.4 rpy=0 -1.13446401 0
- joint right_gripper_joint: limit lower=0.0 upper=0.523599 effort=1000.0 velocity=0.5 -> lower=0.0 upper=0.523599 effort=1000.0 velocity=1.0
