Commit message: "integrated the files and succeeded to induce the robotic model in Gazebo"

File: src/cobrotic/urdf/bak_cobra.urdf (robot description, URDF)
Before this commit: robot cobra, 9 links, 8 joints
Links:
- link left_gripper: geometry visual mesh filename=package://cobrotic/urdf/l_finger.dae
- link left_tip: geometry visual mesh filename=package://cobrotic/urdf/l_finger_tip.dae
- link right_gripper: geometry visual mesh filename=package://cobrotic/urdf/l_finger.dae
- link right_tip: geometry visual mesh filename=package://cobrotic/urdf/l_finger_tip.dae
Joints:
- joint arm_to_forearm: limit lower=0 upper=3.14 effort=1000.0 velocity=1.0 -> lower=0 upper=2.70526034 effort=1000.0 velocity=1.0
- joint bottom_to_pedestal: limit lower=0.00 upper=3.66519143 effort=1000.0 velocity=1.0 -> lower=0.00 upper=3.14 effort=1000.0 velocity=1.0
