Commit message: fixed the order problems of python. Now, it's numerical.

File: install/cobrotic/share/cobrotic/urdf/cobra.urdf (robot description, URDF)
Before this commit: robot cobra, 9 links, 8 joints
Joints:
- joint bottom_to_pedestal: limit lower=0.00 upper=3.14 effort=1000.0 velocity=0.5 -> lower=0.00 upper=3.4906585 effort=1000.0 velocity=0.5

Commit message: "updated a new gripper"

File: install/cobrotic/share/cobrotic/urdf/cobra.urdf (robot description, URDF)
Before this commit: robot cobra, 7 links, 6 joints
Links:
- added link left_point_tip_gripper; collision box size=0.03 0.1 0.1; visual box size=0.03 0.1 0.1
- added link left_tip_gripper; collision box size=0.03 0.1 0.3; visual box size=0.03 0.1 0.3
- added link right_point_tip_gripper; collision box size=0.03 0.1 0.1; visual box size=0.03 0.1 0.1
- added link right_tip_gripper; collision box size=0.03 0.1 0.3; visual box size=0.03 0.1 0.3
- link left_gripper: geometry collision box size=0.03 0.1 0.6; visual box size=0.03 0.1 0.6
- link right_gripper: geometry collision box size=0.03 0.1 0.6; visual box size=0.03 0.1 0.6
Joints:
- added joint left_point_tip_gripper_joint: type fixed, parent left_tip_gripper, child left_point_tip_gripper, origin xyz=0 0 0.25 rpy=0.6 0 0, axis 1 0 0
- added joint left_tip_gripper_joint: type fixed, parent left_gripper, child left_tip_gripper, origin xyz=-0.1 -0.05 0.45 rpy=-0.6 0 0, axis 1 0 0
- added joint right_point_tip_gripper_joint: type fixed, parent right_tip_gripper, child right_point_tip_gripper, origin xyz=0 0 0.25 rpy=-0.6 0 0, axis 1 0 0
- added joint right_tip_gripper_joint: type fixed, parent right_gripper, child right_tip_gripper, origin xyz=-0.1 0.05 0.45 rpy=0.6  0 0, axis 1 0 0
- joint left_gripper_joint: origin xyz=-0.1 -0.08 0.15 rpy=0 0 0 -> xyz=-0.1 -0.15 0.15 rpy=0 0 0
- joint right_gripper_joint: axis 1 0 0 -> -1 0 0; origin xyz=-0.1 0.08 0.15 rpy=0 0 0 -> xyz=-0.1 0.15 0.15 rpy=0 0 0

Commit message: I am going to simulate my robtotic arm to pick up something in Gazebo, so I've decided to commit it before I do that.

File: install/cobrotic/share/cobrotic/urdf/cobra.urdf (robot description, URDF)
Before this commit: robot cobra, 11 links, 10 joints
Links:
- link left_gripper: mass None -> 0.1; geometry collision box size=0.03 0.1 0.3; visual box size=0.03 0.1 0.6
- link left_point_tip_gripper: mass None -> 0.1
- link left_tip_gripper: mass None -> 0.1
- link right_gripper: mass None -> 0.1; geometry collision box size=0.03 0.1 0.3; visual box size=0.03 0.1 0.6
- link right_point_tip_gripper: mass None -> 0.1
- link right_tip_gripper: mass None -> 0.1
Joints:
- joint arm_to_forearm: limit lower=0 upper=2.70526034 effort=1000.0 velocity=1.0 -> lower=0.0 upper=2.70526034 effort=1000.0 velocity=1.0
- joint left_gripper_joint: limit lower=0 upper=0.523599 effort=1000 velocity=1.0 -> lower=0.0 upper=0.523599 effort=1000 velocity=1.0
- joint pedestal_to_arm: limit lower=0 upper=2.18166157 effort=1000.0 velocity=1.0 -> lower=0.0 upper=2.18166157 effort=1000.0 velocity=1.0
- joint right_gripper_joint: limit lower=0 upper=0.523599 effort=1000 velocity=1.0 -> lower=0.0 upper=0.523599 effort=1000 velocity=1.0

Commit message: Successfully published and spawned the controllers.

File: install/cobrotic/share/cobrotic/urdf/cobra.urdf (robot description, URDF)
Before this commit: robot cobra, 11 links, 10 joints
Links:
- added link world
- link arm: mass 4.0 -> 0.3
- link bottom: mass 5.0 -> 1.0
- link forearm: mass 3.0 -> 0.2
- link left_gripper: mass 0.1 -> 0.01
- link left_point_tip_gripper: mass 0.1 -> 0.01
- link left_tip_gripper: mass 0.1 -> 0.01
- link pedestal: mass 3.0 -> 0.2
- link platform: mass 0.5 -> 0.01
- link right_gripper: mass 0.1 -> 0.01
- link right_tip_gripper: mass 0.1 -> 0.01
Joints:
- added joint world_to_bottom: type fixed, parent world, child bottom, origin xyz=0 0 0.3 rpy=0 0 0
- joint bottom_to_pedestal: origin xyz=0 0 0.25 rpy=0 0 0 -> xyz=0 0 0 rpy=0 0 0
